File: board/bbqsensor/bbqsensor.sch (EAGLE design)
At the start: 93 parts, among them IC1 CP2104, J1 B4P-VH, J2 B2P-VH, J3 OSTTH080160, J5 OSTTH080160, J6 AVR_SPI_PRG_6PTH, Q2 mmbt2222, Q5 mmbt2222, Q6 DMG3415U, U1 MAX31850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

Commit message: More documentation
Other:
- note added: "ADC"
- note added: "Buck Converter"
- note added: "Connectors"
- note added: "ESP32"
- note added: "Thermocouple inputs"
- moved on the sheet: 13, 15, 2, 25, 32, 33, CLK, J1-1, J1-2, J1-3, J1-4, J2-1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
